Commit message: adding gripper camera to spot with arm model

File: spot_description/urdf/spot.sensors.gazebo.xacro (robot description, xacro)
@@ -110,4 +110,29 @@
       <xacro:fixed_joint name="camera_back_j" parent="${prefix}base_link" child="${prefix}camera_back" xyz="-0.425 0 0.01" rpy="0 0.3 ${-pi}" />
     </xacro:macro>
+    <!-- Gazebo sensor for gripper camera. The arm_camera_link / arm_camera_optical_frame
+         links are in spot_arm_macro.urdf and exist as TF frames on the real robot too. -->
+    <xacro:macro name="add_arm_camera" params="prefix:='' visualize:=0">
+      <gazebo reference="${prefix}arm_camera_link">
+        <sensor name="arm_camera" type="camera">
+          <pose>0 0 0 0 0 0</pose>
+          <update_rate>30</update_rate>
+          <topic>arm_camera/image</topic>
+          <visualize>${visualize}</visualize>
+          <camera>
+            <horizontal_fov>${radians(90)}</horizontal_fov>
+            <image>
+              <width>640</width>
+              <height>480</height>
+              <format>R8G8B8</format>
+            </image>
+            <clip>
+              <near>0.05</near>
+              <far>10.0</far>
+            </clip>
+            <optical_frame_id>${prefix}arm_camera_optical_frame</optical_frame_id>
+          </camera>
+        </sensor>
+      </gazebo>
+    </xacro:macro>
     <!-- Odometry simulation -->
     <xacro:macro name="spot_odometry_publisher">

File: spot_description/urdf/spot.urdf.xacro (robot description, xacro)
@@ -32,4 +32,5 @@
   <xacro:load_spot
     arm="$(arg arm)"
+    custom_gripper_base_link="palm_link"
     feet="$(arg feet)"
     tf_prefix="$(arg tf_prefix)"
@@ -54,4 +55,9 @@
     <xacro:include filename="$(find spot_description)/urdf/spot.sensors.gazebo.xacro" />
     <xacro:add_cameras prefix="$(arg tf_prefix)" />
+    <xacro:if value="$(arg arm)">
+      <xacro:unless value="$(arg gripperless)">
+        <xacro:add_arm_camera prefix="$(arg tf_prefix)" />
+      </xacro:unless>
+    </xacro:if>
   </xacro:if>
   <!-- Gazebo tags -->

File: spot_description/urdf/spot_macro.xacro (robot description, xacro)
@@ -5,5 +5,5 @@
     feet:=false
     gripperless:=false
-    custom_gripper_base_link:=''
+    custom_gripper_base_link:='palm_link'
     tf_prefix
     include_transmissions=false
